File: 4UBenjolin_Kicad/Benjolin_Kicad.kicad_pcb (KiCad board)
At the start: 2 copper layers, 254 x 177.5 mm, 138 parts, among them J1 Conn_01x03_Female, J10 MAINOUT, J11 PWM, J12 RUN, J13 XOR, J14 CV_1, J15 CV_2, J4 EXT.INPUT, J5 CV_F, J6 PUL2, J7 TRI1, J8 TRI2, J9 PUL1, P10R1 10k, P11R1 10k, P1R1 10k, P2R1 10k, P3R1 10k, P4R1 10k, P5R1 10k, P6R1 10k, P8R1 10k, P9R1 10k, Q1 BC547, SW1 SW_SPDT, U1 TL074, U2 TL072, U3 TL074, U4 TL074, U5 SSI2164, U6 4021, U7 L78L09_SOT89

Commit message: Added footprints and symbols. added a mixer to the panel
Parts:
- removed P10R1, P11R1, P1R1, P2R1, P3R1, P4R1, P5R1, P6R1, P8R1, P9R1: 10k, Potentiometer_THT:Potentiometer_Alps_RK09K_Single_Vertical
- removed REF** (x32): Banana Jack, SynthComponents:Cinch Banana Jack (Panel)
- added C19: 470nf, Capacitor_THT:C_Disc_D8.0mm_W2.5mm_P5.00mm, B.Cu at (185.3, 33.7)
- added C20: 47pf, Capacitor_THT:C_Disc_D8.0mm_W2.5mm_P5.00mm, B.Cu at (231.1, 38.1)
- added C21: 100nf, Capacitor_THT:C_Disc_D8.0mm_W2.5mm_P5.00mm, B.Cu at (205.7, 31.1)
- added J1: Conn_01x04_Male, Connector_Molex:Molex_Micro-Latch_53254-0470_1x04_P2.00mm_Horizontal, B.Cu at (251.6, 160.8)
- added J16: Mix_In_3, SynthComponents:Banana_Jack_PCB, F.Cu at (241.3, 41.3)
- added J17: Mix_In_4, SynthComponents:Banana_Jack_PCB, F.Cu at (266.7, 41.3)
- added J18: Mixer_Out, SynthComponents:Banana_Jack_PCB, F.Cu at (266.7, 22.2)
- added J2: Mix_In_1, SynthComponents:Banana_Jack_PCB, F.Cu at (190.5, 41.3)
- added J3: Mix_In_2, SynthComponents:Banana_Jack_PCB, F.Cu at (215.9, 41.3)
- added P_Chan1: 100k, SynthComponents:Potentiometer_Alps_RK09K_Single_Vertical, F.Cu at (190.5, 22.2)
- added P_Chan2: 100k, SynthComponents:Potentiometer_Alps_RK09K_Single_Vertical, F.Cu at (215.9, 22.2)
- added P_Chan3: 100k, SynthComponents:Potentiometer_Alps_RK09K_Single_Vertical, F.Cu at (241.3, 22.2)
- added P_Filter_Frequency1: 10k, SynthComponents:Potentiometer_Alps_RK09K_Single_Vertical, F.Cu at (241.3, 155.6)
- added P_Filter_Resonance1: 10k, SynthComponents:Potentiometer_Alps_RK09K_Single_Vertical, F.Cu at (266.7, 155.6)
- added P_Freq_A1: 10k, SynthComponents:Potentiometer_Alps_RK09K_Single_Vertical, F.Cu at (190.5, 155.6)
- added P_Freq_B1: 10k, SynthComponents:Potentiometer_Alps_RK09K_Single_Vertical, F.Cu at (215.9, 155.6)
- added P_Mod_A1: 10k, SynthComponents:Potentiometer_Alps_RK09K_Single_Vertical, F.Cu at (190.5, 117.5)
- added P_Mod_B1: 10k, SynthComponents:Potentiometer_Alps_RK09K_Single_Vertical, F.Cu at (215.9, 117.5)
- added P_Mod_Filter1: 10k, SynthComponents:Potentiometer_Alps_RK09K_Single_Vertical, F.Cu at (241.3, 117.5)
- added P_Rungler_A1: 10k, SynthComponents:Potentiometer_Alps_RK09K_Single_Vertical, F.Cu at (190.5, 136.5)
- added P_Rungler_B1: 10k, SynthComponents:Potentiometer_Alps_RK09K_Single_Vertical, F.Cu at (215.9, 136.5)
- added P_Rungler_Filter1: 10k, SynthComponents:Potentiometer_Alps_RK09K_Single_Vertical, F.Cu at (241.3, 136.5)
- added R51: 100K, Resistor_THT:R_Axial_DIN0204_L3.6mm_D1.6mm_P7.62mm_Horizontal, B.Cu at (259.7, 24.8)
- added R52: 100K, Resistor_THT:R_Axial_DIN0204_L3.6mm_D1.6mm_P7.62mm_Horizontal, B.Cu at (259.7, 20.3)
- added R53: 100K, Resistor_THT:R_Axial_DIN0204_L3.6mm_D1.6mm_P7.62mm_Horizontal, B.Cu at (200.7, 16.5)
- added R54: 100K, Resistor_THT:R_Axial_DIN0204_L3.6mm_D1.6mm_P7.62mm_Horizontal, B.Cu at (225.4, 16.5)
- added R55: 100K, Resistor_THT:R_Axial_DIN0204_L3.6mm_D1.6mm_P7.62mm_Horizontal, B.Cu at (259.7, 15.9)
- added R56: 100K, Resistor_THT:R_Axial_DIN0204_L3.6mm_D1.6mm_P7.62mm_Horizontal, B.Cu at (245.1, 32.4)
- added R57: 330R, Resistor_THT:R_Axial_DIN0204_L3.6mm_D1.6mm_P7.62mm_Horizontal, B.Cu at (232.4, 32.4)
- added RV_Loop_Offset1: 10k, SynthComponents:Potentiometer_Alps_RK09K_Single_Vertical, F.Cu at (266.7, 117.5)
- added U8: 79L09, Package_TO_SOT_THT:TO-92L_Inline, B.Cu at (360.7, 143.3)
- added U9: TL071, Package_DIP:DIP-8_W7.62mm_Socket_LongPads, B.Cu at (207.0, 37.5)
- C1, C10, C11, C14, C16, C17, C2, C3, C4, C5, C6, C7, C8, C9: footprint Capacitor_SMD:C_1206_3216Metric_Pad1.42x1.75mm_HandSolder -> Capacitor_THT:C_Disc_D8.0mm_W2.5mm_P5.00mm; moved to B.Cu
- C12, C13, C15, C18, Q1, U7: moved to B.Cu
- D1, D2, D3, D4, D5, D6: footprint Diode_THT:D_DO-35_SOD27_P2.54mm_Vertical_AnodeUp -> Diode_THT:D_A-405_P7.62mm_Horizontal; moved to B.Cu
- J1000: renamed from J1; moved to B.Cu
- R1, R10, R11, R12, R13, R14, R15, R16, R17, R18, R19, R2, R20, R21, R22, R23, R24, R25, R26, R27, R28, R29, R3, R30, R31, R32, R33, R34, R35, R36, R37, R38, R39, R4, R40, R41, R42, R43, R44, R45, R46, R47, R48, R49, R5, R50, R6, R7, R8, R9: footprint Resistor_SMD:R_0603_1608Metric_Pad1.05x0.95mm_HandSolder -> Resistor_THT:R_Axial_DIN0204_L3.6mm_D1.6mm_P7.62mm_Horizontal; moved to B.Cu
- U1, U3, U4: footprint Package_SO:SOIC-14_3.9x8.7mm_P1.27mm -> Package_DIP:DIP-14_W7.62mm_Socket_LongPads; moved to B.Cu
- U2: footprint Package_SO:SOIC-8_3.9x4.9mm_P1.27mm -> Package_DIP:DIP-8_W7.62mm_Socket_LongPads; moved to B.Cu
- U5, U6: footprint Package_SO:SOIC-16_3.9x9.9mm_P1.27mm -> Package_DIP:DIP-16_W7.62mm_Socket_LongPads; moved to B.Cu
- moved R2 207.4 mm to (157.0, 128.0)
- moved R12 204.3 mm to (157.0, 133.1)
- moved R4 193.5 mm to (157.0, 143.3)
- moved R3 185.3 mm to (157.0, 138.2)
- moved D1 183.1 mm to (156.5, 118.4)
- moved U1 179.1 mm to (207.0, 91.4), turned to 180 degrees
- moved D3 155.1 mm to (157.0, 111.3)
- moved U3 138.0 mm to (232.4, 91.4), turned to 180 degrees
- moved R27 120.9 mm to (379.8, 165.2)
- moved SW1 119.4 mm to (266.7, 134.0)
- moved R10 113.6 mm to (355.3, 159.7)
- moved U2 112.4 mm to (207.0, 77.5), turned to 180 degrees
- moved C16 112.2 mm to (399.2, 153.9)
- moved U6 111.7 mm to (207.0, 53.3), turned to 180 degrees
- moved C18 110.5 mm to (422.9, 142.0)
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Connections:
- C14 pad 1: GND -> Net-(C14-Pad1)
- C14 pad 2: V+ -> -12V
- C16 pad 1: Net-(C16-Pad1) -> GND
- C16 pad 2: Net-(C16-Pad2) -> V+
- C17 pad 1: Net-(C17-Pad1) -> Net-(C14-Pad1)
- C18 pad 1: Net-(C18-Pad1) -> Net-(C14-Pad1)
- C18 pad 2: Net-(C18-Pad2) -> Net-(C17-Pad2)
- J1000 pad 1: GND -> Net-(J1000-Pad1)
- J1000 pad 2: +12V -> Net-(J1000-Pad2)
- J1000 pad 3: -12V -> Net-(J1000-Pad3)
Other:
- board text added: "(Rung A)"
- board text added: "(filter freq)"
- board text added: "(filter res)"
- board text added: "(freq A)"
- board text added: "(freq B)"
- board text added: "(loop offset)"
- board text added: "(mod A)"
- board text added: "(mod B)"
- board text added: "(mod Filter)"
- board text added: "(rungler filter)"
- board text added: "CV A"
- board text added: "CV B"
- board text added: "CV1"
- board text added: "Filter CV"
- board text added: "Mix In2"
- board text added: "Mix Out"
- board text added: "MixIn1"
- board text added: "VCA In"
- board text added: "ext. in"
- board text added: "main out"
- board text added: "on/off"
- board text added: "pulse A"
- board text added: "pulse B"
- board text added: "pwm"
- board text added: "rungler"
- board text added: "tri A"
- board text added: "tri B"
- board text added: "xor"

Commit message: Working on board layout
Parts:
- moved R40 189.9 mm to (200.0, 124.5)
- moved R23 183.4 mm to (207.6, 116.8), turned to 180 degrees
- moved R47 182.2 mm to (207.6, 121.9), turned to 180 degrees
- moved C6 179.7 mm to (206.4, 127.6), turned to 180 degrees
- moved R35 175.4 mm to (207.6, 119.4), turned to 180 degrees
- moved C2 173.7 mm to (201.3, 113.7)
- moved R7 166.2 mm to (232.4, 163.2), turned to 180 degrees
- moved C3 165.7 mm to (226.1, 113.7)
- moved R6 162.8 mm to (232.4, 160.5), turned to 180 degrees
- moved R25 154.2 mm to (250.2, 73.0)
- moved R48 151.7 mm to (232.4, 121.9), turned to 180 degrees
- moved R46 151.7 mm to (250.2, 35.6)
- moved R28 151.5 mm to (250.2, 82.5)
- moved D2 150.5 mm to (224.8, 152.4)
- moved R27 149.9 mm to (257.8, 78.1), turned to 180 degrees
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
Commit message: ready for traces
Parts:
- moved R9 181.3 mm to (186.7, 88.9)
- moved R45 180.4 mm to (250.2, 121.3)
- moved R37 170.5 mm to (257.8, 108.6), turned to 180 degrees
- moved C18 163.9 mm to (259.1, 139.7)
- moved R8 163.9 mm to (257.8, 128.9), turned to 180 degrees
- moved C16 151.3 mm to (275.6, 66.7), turned to 270 degrees
- moved R49 150.1 mm to (250.2, 111.1)
- moved R39 149.8 mm to (257.8, 123.8), turned to 180 degrees
- moved C15 148.8 mm to (266.1, 128.2), turned to 90 degrees
- moved C13 148.0 mm to (254.6, 139.7), turned to 180 degrees
- moved R43 141.6 mm to (250.2, 113.7)
- moved C12 141.1 mm to (252.1, 147.3)
- moved C11 132.0 mm to (275.6, 81.9), turned to 90 degrees
- moved R15 123.7 mm to (250.2, 126.4)
- moved R38 123.4 mm to (250.2, 116.2)
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
Commit message: traces complete
Parts:
- removed J1000: Conn_01x03_Female, Connector_PinSocket_2.54mm:PinSocket_1x03_P2.54mm_Vertical
- added REF**: Banana Jack, SynthComponents:Banana _Jack_Panel, F.Cu at (117.5, 109.5)
- added REF**: Banana Jack, SynthComponents:Banana _Jack_Panel, F.Cu at (92.1, 71.4)
- added REF**: Banana Jack, SynthComponents:Banana _Jack_Panel, F.Cu at (66.7, 71.4)
- added REF**: Banana Jack, SynthComponents:Banana _Jack_Panel, F.Cu at (41.3, 71.4)
- added REF**: Banana Jack, SynthComponents:Banana _Jack_Panel, F.Cu at (41.3, 52.4)
- added REF**: Banana Jack, SynthComponents:Banana _Jack_Panel, F.Cu at (66.7, 52.4)
- added REF**: Banana Jack, SynthComponents:Banana _Jack_Panel, F.Cu at (92.1, 52.4)
- added REF**: Banana Jack, SynthComponents:Banana _Jack_Panel, F.Cu at (117.5, 52.4)
- added REF**: Banana Jack, SynthComponents:Banana _Jack_Panel, F.Cu at (117.5, 33.3)
- added REF**: Banana Jack, SynthComponents:Banana _Jack_Panel, F.Cu at (92.1, 109.5)
- added REF**: Banana Jack, SynthComponents:Banana _Jack_Panel, F.Cu at (66.7, 109.5)
- added REF**: Banana Jack, SynthComponents:Banana _Jack_Panel, F.Cu at (41.3, 109.5)
- added REF**: Banana Jack, SynthComponents:Banana _Jack_Panel, F.Cu at (41.3, 90.5)
- added REF**: Banana Jack, SynthComponents:Banana _Jack_Panel, F.Cu at (66.7, 90.5)
- added REF**: Banana Jack, SynthComponents:Banana _Jack_Panel, F.Cu at (92.1, 90.5)
- added REF**: Banana Jack, SynthComponents:Banana _Jack_Panel, F.Cu at (117.5, 90.5)
- added REF**: Banana Jack, SynthComponents:Banana _Jack_Panel, F.Cu at (117.5, 71.4)
- moved R9 85.2 mm to (262.9, 127.0)
- moved C11 81.5 mm to (269.2, 163.2), turned to 180 degrees
- moved U5 73.0 mm to (232.4, 118.1)
- moved C16 63.3 mm to (256.5, 127.0), turned to 180 degrees
- moved U7 55.4 mm to (250.8, 140.3), turned to 270 degrees
- moved R27 52.7 mm to (257.8, 25.4)
- moved D1 52.1 mm to (199.4, 100.3)
- moved D3 52.1 mm to (199.4, 96.5)
- moved R3 52.1 mm to (207.0, 108.6)
- moved R4 52.1 mm to (207.0, 106.0)
- moved R12 52.1 mm to (199.4, 103.5)
- moved R2 52.1 mm to (207.0, 111.1)
- moved C4 51.2 mm to (256.5, 19.7), turned to 180 degrees
- moved R25 50.2 mm to (250.2, 22.9)
- moved C8 48.7 mm to (205.7, 79.4)
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Connections:
- P_Filter_Resonance1 pad 3: P9R3F -> P9R3B
Routing:
- net V+: track 0.00 -> 366.9 mm, vias 0 -> 10
- net V-: track 0.00 -> 363.6 mm, vias 0 -> 12
- net RUN_CV: track 0.00 -> 216.6 mm, vias 0 -> 8
- net Net-(C5-Pad1): track 0.00 -> 186.2 mm, vias 0 -> 5
- net P2: track 0.00 -> 185.5 mm, vias 0 -> 2
- net P9R2B: track 0.00 -> 160.1 mm
- net P9R3B: track 0.00 -> 150.6 mm, vias 0 -> 6
- net T2: track 0.00 -> 144.2 mm, vias 0 -> 1
- net P1: track 0.00 -> 140.2 mm, vias 0 -> 7
- net VCA2In: track 0.00 -> 131.5 mm
- net Net-(Q1-Pad1): track 0.00 -> 128.7 mm, vias 0 -> 4
- net XOR: track 0.00 -> 113.0 mm, vias 0 -> 6
- net Net-(R15-Pad1): track 0.00 -> 109.3 mm
- net T1: track 0.00 -> 102.9 mm, vias 0 -> 5
- net Net-(D5-Pad1): track 0.00 -> 100.4 mm, vias 0 -> 5
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- added copper zone on B.Cu, net GND
- added copper zone on F.Cu, net GND
Other:
- outline, holes or cut-outs redrawn

Commit message: fixed banana panel cutout, designed front panel for Benjolin, Fixed pot orientation
Parts:
- moved SW1 5.08 mm to (266.7, 139.1), turned to 180 degrees
Connections:
- P_Chan1 pad 1: Net-(J2-Pad1) -> GND
- P_Chan1 pad 3: GND -> Net-(J2-Pad1)
- P_Chan2 pad 1: Net-(J3-Pad1) -> GND
- P_Chan2 pad 3: GND -> Net-(J3-Pad1)
- P_Chan3 pad 1: Net-(J16-Pad1) -> GND
- P_Chan3 pad 3: GND -> Net-(J16-Pad1)
- P_Filter_Resonance1 pad 1: GND -> P9R3B
- P_Filter_Resonance1 pad 3: P9R3B -> GND
- P_Mod_A1 pad 1: Net-(J14-Pad1) -> GND
- P_Mod_A1 pad 3: GND -> Net-(J14-Pad1)
- P_Mod_B1 pad 1: Net-(J15-Pad1) -> GND
- P_Mod_B1 pad 3: GND -> Net-(J15-Pad1)
- P_Mod_Filter1 pad 1: Net-(J5-Pad1) -> GND
- P_Mod_Filter1 pad 3: GND -> Net-(J5-Pad1)
- P_Rungler_A1 pad 1: RUN_CV -> GND
- P_Rungler_A1 pad 3: GND -> RUN_CV
- P_Rungler_B1 pad 1: RUN_CV -> GND
- P_Rungler_B1 pad 3: GND -> RUN_CV
- P_Rungler_Filter1 pad 1: RUN_CV -> GND
- P_Rungler_Filter1 pad 3: GND -> RUN_CV
- RV_Loop_Offset1 pad 1: V+ -> V-
- RV_Loop_Offset1 pad 3: V- -> V+
Routing:
- net P9R3B: track 150.6 -> 158.9 mm
- net V+: track 366.9 -> 374.2 mm
- net Net-(R1-Pad2): track 11.1 -> 17.4 mm
- net V-: track 363.6 -> 358.7 mm, vias 12 -> 13
- net GND: track 27.0 -> 22.3 mm, vias 127 -> 130
- net Net-(J2-Pad1): track 20.8 -> 18.7 mm
- net RUN_CV: track 216.6 -> 214.9 mm, vias 8 -> 7
- net P1R2B: track 10.5 -> 11.6 mm
- net Net-(J3-Pad1): track 27.1 -> 26.8 mm, vias 0 -> 1
Other:
- board size 254 x 177.5 mm -> 254 x 177.8 mm
- board text added: "BENJOLIN AND MIXER"
- board text added: "CV"
- board text added: "EXT. IN"
- board text added: "FILTER FREQ"
- board text added: "FREQ A"
- board text added: "FREQ B"
- board text added: "IN 1"
- board text added: "IN 2"
- board text added: "IN 3"
- board text added: "IN 4"
- board text added: "LOOP OFFSET"
- board text added: "MAIN OUT"
- board text added: "MIX OUT"
- board text added: "ON/OFF"
- board text added: "PULSE"
- board text added: "PWM"
- board text added: "RESONANCE"
- board text added: "RUNGLER"
- board text added: "RUNGLER CV"
- board text added: "TRIANGLE"
- board text added: "XOR"
- board text removed: "(Rung A)"
- board text removed: "(filter freq)"
- board text removed: "(filter res)"
- board text removed: "(freq A)"
- board text removed: "(freq B)"
- board text removed: "(loop offset)"
- board text removed: "(mod A)"
- board text removed: "(mod B)"
- board text removed: "(mod Filter)"
- board text removed: "(rungler filter)"
- board text removed: "CV A"
- board text removed: "CV B"
- board text removed: "CV1"
- board text removed: "Filter CV"
- board text removed: "Mix In2"
- board text removed: "Mix Out"
- board text removed: "MixIn1"
- board text removed: "VCA In"
- board text removed: "ext. in"
- board text removed: "main out"
- board text removed: "on/off"
- board text removed: "pulse A"
- board text removed: "pulse B"
- board text removed: "pwm"
- board text removed: "rungler"
- board text removed: "tri A"
- board text removed: "tri B"
- board text removed: "xor"

Commit message: worked on front panel
Other:
- board text added: "LOOP I/Ø"
- board text removed: "ON/OFF"
Changed lines of the file:
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@@
   )
   (setup
-    (last_trace_width 0.508)
+    (last_trace_width 0.25)
     (user_trace_width 0.381)
     (user_trace_width 0.508)
@@
     (effects (font (size 2 2) (thickness 0.5)))
   )
-  (gr_text ON/OFF (at 117.475 156.21) (layer F.Cu)
+  (gr_text "LOOP I/Ø" (at 117.475 156.21) (layer F.Cu)
     (effects (font (size 2 2) (thickness 0.5)))
   )
